File: kicad/buffer_ram_sch.kicad_sch (KiCad schematic)
At the start: 6 parts, among them U12 HM6264LP, U13 HM6264LP, U14 74LS02

Commit message: KiCAD: Initial PCB placement
Parts:
- R1, R2, R3: footprint (none) -> custom_footprints:R_Axial_DIN0207_L6.3mm_D2.0mm_P10.16mm_Horizontal
- U12, U13: footprint Package_DIP:DIP-28_W15.24mm -> Package_DIP:DIP-28_W15.24mm_LongPads
- U14: footprint (none) -> Package_DIP:DIP-14_W7.62mm_LongPads
Changed lines of the file:
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@@
       (effects (font (size 1.27 1.27)) (justify left))
     )
-    (property "Footprint" "Package_DIP:DIP-28_W15.24mm" (id 2) (at 224.79 93.98 0)
+    (property "Footprint" "Package_DIP:DIP-28_W15.24mm_LongPads" (id 2) (at 224.79 93.98 0)
       (effects (font (size 1.27 1.27)) hide)
     )
@@
       (effects (font (size 1.27 1.27)) (justify left))
     )
-    (property "Footprint" "" (id 2) (at 96.012 110.49 90)
+    (property "Footprint" "custom_footprints:R_Axial_DIN0207_L6.3mm_D2.0mm_P10.16mm_Horizontal" (id 2) (at 96.012 110.49 90)
       (effects (font (size 1.27 1.27)) hide)
     )
@@
       (effects (font (size 1.27 1.27)) (justify left))
     )
-    (property "Footprint" "Package_DIP:DIP-28_W15.24mm" (id 2) (at 166.37 93.98 0)
+    (property "Footprint" "Package_DIP:DIP-28_W15.24mm_LongPads" (id 2) (at 166.37 93.98 0)
       (effects (font (size 1.27 1.27)) hide)
     )
@@
       (effects (font (size 1.27 1.27)) (justify left))
     )
-    (property "Footprint" "" (id 2) (at 116.332 110.49 90)
+    (property "Footprint" "custom_footprints:R_Axial_DIN0207_L6.3mm_D2.0mm_P10.16mm_Horizontal" (id 2) (at 116.332 110.49 90)
       (effects (font (size 1.27 1.27)) hide)
     )
@@
     (property "Reference" "U14" (id 0) (at 214.63 133.35 0))
     (property "Value" "74LS02" (id 1) (at 214.63 135.89 0))
-    (property "Footprint" "" (id 2) (at 214.63 142.24 0)
+    (property "Footprint" "Package_DIP:DIP-14_W7.62mm_LongPads" (id 2) (at 214.63 142.24 0)
       (effects (font (size 1.27 1.27)) hide)
     )
@@
       (effects (font (size 1.27 1.27)) (justify left))
     )
-    (property "Footprint" "" (id 2) (at 106.172 110.49 90)
-      (effects (font (size 1.27 1.27)) hide)
-    )
+    (property "Footprint" "custom_footprints:R_Axial_DIN0207_L6.3mm_D2.0mm_P10.16mm_Horizontal" (id 2) (at 106.172 110.49 90)
+      (effects (font (size 1.27 1.27)) hide)
+    )

Commit message: KiCAD: PCB now routed
Parts:
- U12, U13: footprint Package_DIP:DIP-28_W15.24mm_LongPads -> Package_DIP:DIP-28_W15.24mm
- U14: footprint Package_DIP:DIP-14_W7.62mm_LongPads -> Package_DIP:DIP-14_W7.62mm
Connections:
- net nAddr13: now reaches U13.26 (CE2), U14.1
Changed lines of the file:
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@@
+    (effects (font (size 1.27 1.27)) (justify left bottom))
+  )
+  (label "nAddr13" (at 231.14 142.24 0)
     (effects (font (size 1.27 1.27)) (justify left bottom))
   )
@@
       (effects (font (size 1.27 1.27)) (justify left))
     )
-    (property "Footprint" "Package_DIP:DIP-28_W15.24mm_LongPads" (id 2) (at 224.79 93.98 0)
+    (property "Footprint" "Package_DIP:DIP-28_W15.24mm" (id 2) (at 224.79 93.98 0)
       (effects (font (size 1.27 1.27)) hide)
     )
@@
       (effects (font (size 1.27 1.27)) (justify left))
     )
-    (property "Footprint" "Package_DIP:DIP-28_W15.24mm_LongPads" (id 2) (at 166.37 93.98 0)
+    (property "Footprint" "Package_DIP:DIP-28_W15.24mm" (id 2) (at 166.37 93.98 0)
       (effects (font (size 1.27 1.27)) hide)
     )
@@
     (property "Reference" "U14" (id 0) (at 214.63 133.35 0))
     (property "Value" "74LS02" (id 1) (at 214.63 135.89 0))
-    (property "Footprint" "Package_DIP:DIP-14_W7.62mm_LongPads" (id 2) (at 214.63 142.24 0)
+    (property "Footprint" "Package_DIP:DIP-14_W7.62mm" (id 2) (at 214.63 142.24 0)
       (effects (font (size 1.27 1.27)) hide)
     )

Commit message: KiCAD - more silk screen
Parts:
- U12, U13: footprint Package_DIP:DIP-28_W15.24mm -> Package_DIP:DIP-28_W15.24mm_Socket
- U14: footprint Package_DIP:DIP-14_W7.62mm -> Package_DIP:DIP-14_W7.62mm_Socket
Changed lines of the file:
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@@
       (effects (font (size 1.27 1.27)) (justify left))
     )
-    (property "Footprint" "Package_DIP:DIP-28_W15.24mm" (id 2) (at 224.79 93.98 0)
+    (property "Footprint" "Package_DIP:DIP-28_W15.24mm_Socket" (id 2) (at 224.79 93.98 0)
       (effects (font (size 1.27 1.27)) hide)
     )
@@
       (effects (font (size 1.27 1.27)) (justify left))
     )
-    (property "Footprint" "Package_DIP:DIP-28_W15.24mm" (id 2) (at 166.37 93.98 0)
+    (property "Footprint" "Package_DIP:DIP-28_W15.24mm_Socket" (id 2) (at 166.37 93.98 0)
       (effects (font (size 1.27 1.27)) hide)
     )
@@
     (property "Reference" "U14" (id 0) (at 214.63 133.35 0))
     (property "Value" "74LS02" (id 1) (at 214.63 135.89 0))
-    (property "Footprint" "Package_DIP:DIP-14_W7.62mm" (id 2) (at 214.63 142.24 0)
+    (property "Footprint" "Package_DIP:DIP-14_W7.62mm_Socket" (id 2) (at 214.63 142.24 0)
       (effects (font (size 1.27 1.27)) hide)
     )

Commit message: KiCAD: Customize IC footprint silk screen
Parts:
- U12, U13: footprint Package_DIP:DIP-28_W15.24mm_Socket -> custom_footprints:DIP-28_W15.24mm_Socket
- U14: footprint Package_DIP:DIP-14_W7.62mm_Socket -> custom_footprints:DIP-14_W7.62mm_Socket
Changed lines of the file:
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@@
       (effects (font (size 1.27 1.27)) (justify left))
     )
-    (property "Footprint" "Package_DIP:DIP-28_W15.24mm_Socket" (id 2) (at 224.79 93.98 0)
+    (property "Footprint" "custom_footprints:DIP-28_W15.24mm_Socket" (id 2) (at 224.79 93.98 0)
       (effects (font (size 1.27 1.27)) hide)
     )
@@
       (effects (font (size 1.27 1.27)) (justify left))
     )
-    (property "Footprint" "Package_DIP:DIP-28_W15.24mm_Socket" (id 2) (at 166.37 93.98 0)
+    (property "Footprint" "custom_footprints:DIP-28_W15.24mm_Socket" (id 2) (at 166.37 93.98 0)
       (effects (font (size 1.27 1.27)) hide)
     )
@@
     (property "Reference" "U14" (id 0) (at 214.63 133.35 0))
     (property "Value" "74LS02" (id 1) (at 214.63 135.89 0))
-    (property "Footprint" "Package_DIP:DIP-14_W7.62mm_Socket" (id 2) (at 214.63 142.24 0)
+    (property "Footprint" "custom_footprints:DIP-14_W7.62mm_Socket" (id 2) (at 214.63 142.24 0)
       (effects (font (size 1.27 1.27)) hide)
     )
