File: kicad/main_logic.kicad_sch (KiCad schematic)
At the start: 14 parts, among them U10 74LS00, U17 28 PIN ZIF, U3 74LS245, U4 74LS244, U5 74LS244, U8 74LS04, U9 74LS08

Commit message: Fixed following stardot discussion of PSU, and review of issue 2 photos
Parts:
- R4: value 1K0 -> 3K3
Changed lines of the file:
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@@
       (effects (font (size 1.27 1.27)) (justify left))
     )
-    (property "Value" "1K0" (id 1) (at 154.94 97.7899 0)
+    (property "Value" "3K3" (id 1) (at 154.94 97.7899 0)
       (effects (font (size 1.27 1.27)) (justify left))
     )

Commit message: KiCAD: Initial PCB placement
Parts:
- D1, D2, D3: footprint (none) -> custom_footprints:D_DO-35_SOD27_P11.43mm_Horizontal
- R4: footprint (none) -> custom_footprints:R_Axial_DIN0207_L6.3mm_D2.0mm_P11.43mm_Horizontal
- RL1, RL2, RL3: footprint Relay_THT:Relay_DPDT_Omron_G2RL -> Relay_THT:Relay_DPDT_Omron_G5V-2
- U10, U8, U9: footprint (none) -> Package_DIP:DIP-14_W7.62mm_LongPads
- U17: footprint Package_DIP:DIP-28_W15.24mm -> Package_DIP:DIP-28_W15.24mm_Socket_LongPads
- U3, U4, U5: footprint (none) -> Package_DIP:DIP-20_W7.62mm_LongPads
Changed lines of the file:
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@@
     (property "Reference" "U10" (id 0) (at 78.74 73.66 0))
     (property "Value" "74LS00" (id 1) (at 78.74 76.2 0))
-    (property "Footprint" "" (id 2) (at 78.74 82.55 0)
+    (property "Footprint" "Package_DIP:DIP-14_W7.62mm_LongPads" (id 2) (at 78.74 82.55 0)
       (effects (font (size 1.27 1.27)) hide)
     )
@@
     (property "Reference" "U9" (id 0) (at 41.91 153.67 0))
     (property "Value" "74LS08" (id 1) (at 41.91 156.21 0))
-    (property "Footprint" "" (id 2) (at 41.91 161.29 0)
+    (property "Footprint" "Package_DIP:DIP-14_W7.62mm_LongPads" (id 2) (at 41.91 161.29 0)
       (effects (font (size 1.27 1.27)) hide)
     )
@@
     (property "Reference" "D3" (id 0) (at 179.07 119.38 0))
     (property "Value" "1N4148" (id 1) (at 185.42 119.38 0))
-    (property "Footprint" "" (id 2) (at 181.61 116.84 0)
+    (property "Footprint" "custom_footprints:D_DO-35_SOD27_P11.43mm_Horizontal" (id 2) (at 181.61 116.84 0)
       (effects (font (size 1.27 1.27)) hide)
     )
@@
     (property "Reference" "D2" (id 0) (at 220.98 151.13 0))
     (property "Value" "1N4148" (id 1) (at 214.63 151.13 0))
-    (property "Footprint" "" (id 2) (at 218.44 148.59 0)
+    (property "Footprint" "custom_footprints:D_DO-35_SOD27_P11.43mm_Horizontal" (id 2) (at 218.44 148.59 0)
       (effects (font (size 1.27 1.27)) hide)
     )
@@
       (effects (font (size 1.27 1.27)) (justify left))
     )
-    (property "Footprint" "" (id 2) (at 80.01 167.64 0)
+    (property "Footprint" "Package_DIP:DIP-14_W7.62mm_LongPads" (id 2) (at 80.01 167.64 0)
       (effects (font (size 1.27 1.27)) hide)
     )
@@
     (property "Reference" "RL2" (id 0) (at 218.44 111.76 90))
     (property "Value" "MT2-C93401" (id 1) (at 218.44 114.3 90))
-    (property "Footprint" "Relay_THT:Relay_DPDT_Omron_G2RL" (id 2) (at 217.17 114.3 0)
+    (property "Footprint" "Relay_THT:Relay_DPDT_Omron_G5V-2" (id 2) (at 217.17 114.3 0)
       (effects (font (size 1.27 1.27)) (justify left) hide)
     )
@@
     (property "Reference" "U8" (id 0) (at 57.15 146.685 0))
     (property "Value" "74LS04" (id 1) (at 57.15 149.225 0))
-    (property "Footprint" "" (id 2) (at 57.15 154.94 0)
+    (property "Footprint" "Package_DIP:DIP-14_W7.62mm_LongPads" (id 2) (at 57.15 154.94 0)
       (effects (font (size 1.27 1.27)) hide)
     )
@@
     (property "Reference" "U10" (id 0) (at 63.5 82.55 0))
     (property "Value" "74LS00" (id 1) (at 63.5 85.09 0))
-    (property "Footprint" "" (id 2) (at 63.5 91.44 0)
+    (property "Footprint" "Package_DIP:DIP-14_W7.62mm_LongPads" (id 2) (at 63.5 91.44 0)
       (effects (font (size 1.27 1.27)) hide)
     )
@@
       (effects (font (size 1.27 1.27)) (justify left))
     )
-    (property "Footprint" "" (id 2) (at 100.33 167.64 0)
+    (property "Footprint" "Package_DIP:DIP-14_W7.62mm_LongPads" (id 2) (at 100.33 167.64 0)
       (effects (font (size 1.27 1.27)) hide)
     )
@@
     (property "Reference" "U8" (id 0) (at 48.26 80.645 0))
     (property "Value" "74LS04" (id 1) (at 48.26 83.185 0))
-    (property "Footprint" "" (id 2) (at 48.26 88.9 0)
+    (property "Footprint" "Package_DIP:DIP-14_W7.62mm_LongPads" (id 2) (at 48.26 88.9 0)
       (effects (font (size 1.27 1.27)) hide)
     )
@@
     (property "Reference" "U10" (id 0) (at 63.5 66.04 0))
     (property "Value" "74LS00" (id 1) (at 63.5 68.58 0))
-    (property "Footprint" "" (id 2) (at 63.5 74.93 0)
+    (property "Footprint" "Package_DIP:DIP-14_W7.62mm_LongPads" (id 2) (at 63.5 74.93 0)
       (effects (font (size 1.27 1.27)) hide)
     )
@@
       (effects (font (size 1.27 1.27)) (justify left))
     )
-    (property "Footprint" "" (id 2) (at 124.46 54.61 0)
+    (property "Footprint" "Package_DIP:DIP-20_W7.62mm_LongPads" (id 2) (at 124.46 54.61 0)
       (effects (font (size 1.27 1.27)) hide)
     )
@@
       (effects (font (size 1.27 1.27)) (justify left))
     )
-    (property "Footprint" "Package_DIP:DIP-28_W15.24mm" (id 2) (at 222.25 64.77 0)
+    (property "Footprint" "Package_DIP:DIP-28_W15.24mm_Socket_LongPads" (id 2) (at 222.25 64.77 0)
       (effects (font (size 1.27 1.27)) hide)
     )
@@
     (property "Reference" "RL1" (id 0) (at 181.61 121.92 90))
     (property "Value" "MT2-C93401" (id 1) (at 181.61 124.46 90))
-    (property "Footprint" "Relay_THT:Relay_DPDT_Omron_G2RL" (id 2) (at 182.88 124.46 0)
+    (property "Footprint" "Relay_THT:Relay_DPDT_Omron_G5V-2" (id 2) (at 182.88 124.46 0)
       (effects (font (size 1.27 1.27)) (justify left) hide)
     )
@@
       (effects (font (size 1.27 1.27)) (justify left))
     )
-    (property "Footprint" "" (id 2) (at 256.54 54.61 0)
+    (property "Footprint" "Package_DIP:DIP-20_W7.62mm_LongPads" (id 2) (at 256.54 54.61 0)
       (effects (font (size 1.27 1.27)) hide)
     )
@@
     (property "Reference" "U8" (id 0) (at 57.15 160.655 0))
     (property "Value" "74LS04" (id 1) (at 57.15 163.195 0))
-    (property "Footprint" "" (id 2) (at 57.15 168.91 0)
+    (property "Footprint" "Package_DIP:DIP-14_W7.62mm_LongPads" (id 2) (at 57.15 168.91 0)
       (effects (font (size 1.27 1.27)) hide)
     )
@@
     (property "Reference" "U10" (id 0) (at 41.91 167.64 0))
     (property "Value" "74LS00" (id 1) (at 41.91 170.18 0))
-    (property "Footprint" "" (id 2) (at 41.91 176.53 0)
+    (property "Footprint" "Package_DIP:DIP-14_W7.62mm_LongPads" (id 2) (at 41.91 176.53 0)
       (effects (font (size 1.27 1.27)) hide)
     )
@@
       (effects (font (size 1.27 1.27)) (justify left))
     )
-    (property "Footprint" "" (id 2) (at 120.65 167.64 0)
+    (property "Footprint" "Package_DIP:DIP-14_W7.62mm_LongPads" (id 2) (at 120.65 167.64 0)
       (effects (font (size 1.27 1.27)) hide)
     )
@@
       (effects (font (size 1.27 1.27)) (justify left))
     )
-    (property "Footprint" "" (id 2) (at 124.46 109.22 0)
+    (property "Footprint" "Package_DIP:DIP-20_W7.62mm_LongPads" (id 2) (at 124.46 109.22 0)
       (effects (font (size 1.27 1.27)) hide)
     )
@@
     (property "Reference" "U8" (id 0) (at 57.15 174.625 0))
     (property "Value" "74LS04" (id 1) (at 57.15 177.165 0))
-    (property "Footprint" "" (id 2) (at 57.15 182.88 0)
+    (property "Footprint" "Package_DIP:DIP-14_W7.62mm_LongPads" (id 2) (at 57.15 182.88 0)
       (effects (font (size 1.27 1.27)) hide)
     )
@@
     (property "Reference" "U9" (id 0) (at 63.5 99.06 0))
     (property "Value" "74LS08" (id 1) (at 63.5 101.6 0))
-    (property "Footprint" "" (id 2) (at 63.5 106.68 0)
+    (property "Footprint" "Package_DIP:DIP-14_W7.62mm_LongPads" (id 2) (at 63.5 106.68 0)
       (effects (font (size 1.27 1.27)) hide)
     )
@@
       (effects (font (size 1.27 1.27)) (justify left))
     )
-    (property "Footprint" "" (id 2) (at 159.258 96.52 90)
+    (property "Footprint" "custom_footprints:R_Axial_DIN0207_L6.3mm_D2.0mm_P11.43mm_Horizontal" (id 2) (at 159.258 96.52 90)
       (effects (font (size 1.27 1.27)) hide)
     )
@@
     (property "Reference" "RL3" (id 0) (at 181.61 80.01 90))
     (property "Value" "MT2-C93401" (id 1) (at 181.61 82.55 90))
-    (property "Footprint" "Relay_THT:Relay_DPDT_Omron_G2RL" (id 2) (at 182.88 82.55 0)
+    (property "Footprint" "Relay_THT:Relay_DPDT_Omron_G5V-2" (id 2) (at 182.88 82.55 0)
       (effects (font (size 1.27 1.27)) (justify left) hide)
     )
@@
     (property "Reference" "D1" (id 0) (at 179.07 161.29 0))
     (property "Value" "1N4148" (id 1) (at 185.42 161.29 0))
-    (property "Footprint" "" (id 2) (at 181.61 158.75 0)
-      (effects (font (size 1.27 1.27)) hide)
-    )
+    (property "Footprint" "custom_footprints:D_DO-35_SOD27_P11.43mm_Horizontal" (id 2) (at 181.61 158.75 0)
+      (effects (font (size 1.27 1.27)) hide)
+    )

Commit message: KiCAD: PCB now routed
Parts:
- U10, U8, U9: footprint Package_DIP:DIP-14_W7.62mm_LongPads -> Package_DIP:DIP-14_W7.62mm
- U17: footprint Package_DIP:DIP-28_W15.24mm_Socket_LongPads -> Package_DIP:DIP-28_W15.24mm_Socket
- U3, U4, U5: footprint Package_DIP:DIP-20_W7.62mm_LongPads -> Package_DIP:DIP-20_W7.62mm
Changed lines of the file:
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@@
     (property "Reference" "U10" (id 0) (at 78.74 73.66 0))
     (property "Value" "74LS00" (id 1) (at 78.74 76.2 0))
-    (property "Footprint" "Package_DIP:DIP-14_W7.62mm_LongPads" (id 2) (at 78.74 82.55 0)
+    (property "Footprint" "Package_DIP:DIP-14_W7.62mm" (id 2) (at 78.74 82.55 0)
       (effects (font (size 1.27 1.27)) hide)
     )
@@
     (property "Reference" "U9" (id 0) (at 41.91 153.67 0))
     (property "Value" "74LS08" (id 1) (at 41.91 156.21 0))
-    (property "Footprint" "Package_DIP:DIP-14_W7.62mm_LongPads" (id 2) (at 41.91 161.29 0)
+    (property "Footprint" "Package_DIP:DIP-14_W7.62mm" (id 2) (at 41.91 161.29 0)
       (effects (font (size 1.27 1.27)) hide)
     )
@@
       (effects (font (size 1.27 1.27)) (justify left))
     )
-    (property "Footprint" "Package_DIP:DIP-14_W7.62mm_LongPads" (id 2) (at 80.01 167.64 0)
+    (property "Footprint" "Package_DIP:DIP-14_W7.62mm" (id 2) (at 80.01 167.64 0)
       (effects (font (size 1.27 1.27)) hide)
     )
@@
     (property "Reference" "U8" (id 0) (at 57.15 146.685 0))
     (property "Value" "74LS04" (id 1) (at 57.15 149.225 0))
-    (property "Footprint" "Package_DIP:DIP-14_W7.62mm_LongPads" (id 2) (at 57.15 154.94 0)
+    (property "Footprint" "Package_DIP:DIP-14_W7.62mm" (id 2) (at 57.15 154.94 0)
       (effects (font (size 1.27 1.27)) hide)
     )
@@
     (property "Reference" "U10" (id 0) (at 63.5 82.55 0))
     (property "Value" "74LS00" (id 1) (at 63.5 85.09 0))
-    (property "Footprint" "Package_DIP:DIP-14_W7.62mm_LongPads" (id 2) (at 63.5 91.44 0)
+    (property "Footprint" "Package_DIP:DIP-14_W7.62mm" (id 2) (at 63.5 91.44 0)
       (effects (font (size 1.27 1.27)) hide)
     )
@@
       (effects (font (size 1.27 1.27)) (justify left))
     )
-    (property "Footprint" "Package_DIP:DIP-14_W7.62mm_LongPads" (id 2) (at 100.33 167.64 0)
+    (property "Footprint" "Package_DIP:DIP-14_W7.62mm" (id 2) (at 100.33 167.64 0)
       (effects (font (size 1.27 1.27)) hide)
     )
@@
     (property "Reference" "U8" (id 0) (at 48.26 80.645 0))
     (property "Value" "74LS04" (id 1) (at 48.26 83.185 0))
-    (property "Footprint" "Package_DIP:DIP-14_W7.62mm_LongPads" (id 2) (at 48.26 88.9 0)
+    (property "Footprint" "Package_DIP:DIP-14_W7.62mm" (id 2) (at 48.26 88.9 0)
       (effects (font (size 1.27 1.27)) hide)
     )
@@
     (property "Reference" "U10" (id 0) (at 63.5 66.04 0))
     (property "Value" "74LS00" (id 1) (at 63.5 68.58 0))
-    (property "Footprint" "Package_DIP:DIP-14_W7.62mm_LongPads" (id 2) (at 63.5 74.93 0)
+    (property "Footprint" "Package_DIP:DIP-14_W7.62mm" (id 2) (at 63.5 74.93 0)
       (effects (font (size 1.27 1.27)) hide)
     )
@@
       (effects (font (size 1.27 1.27)) (justify left))
     )
-    (property "Footprint" "Package_DIP:DIP-20_W7.62mm_LongPads" (id 2) (at 124.46 54.61 0)
+    (property "Footprint" "Package_DIP:DIP-20_W7.62mm" (id 2) (at 124.46 54.61 0)
       (effects (font (size 1.27 1.27)) hide)
     )
@@
       (effects (font (size 1.27 1.27)) (justify left))
     )
-    (property "Footprint" "Package_DIP:DIP-28_W15.24mm_Socket_LongPads" (id 2) (at 222.25 64.77 0)
+    (property "Footprint" "Package_DIP:DIP-28_W15.24mm_Socket" (id 2) (at 222.25 64.77 0)
       (effects (font (size 1.27 1.27)) hide)
     )
@@
       (effects (font (size 1.27 1.27)) (justify left))
     )
-    (property "Footprint" "Package_DIP:DIP-20_W7.62mm_LongPads" (id 2) (at 256.54 54.61 0)
+    (property "Footprint" "Package_DIP:DIP-20_W7.62mm" (id 2) (at 256.54 54.61 0)
       (effects (font (size 1.27 1.27)) hide)
     )
@@
     (property "Reference" "U8" (id 0) (at 57.15 160.655 0))
     (property "Value" "74LS04" (id 1) (at 57.15 163.195 0))
-    (property "Footprint" "Package_DIP:DIP-14_W7.62mm_LongPads" (id 2) (at 57.15 168.91 0)
+    (property "Footprint" "Package_DIP:DIP-14_W7.62mm" (id 2) (at 57.15 168.91 0)
       (effects (font (size 1.27 1.27)) hide)
     )
@@
     (property "Reference" "U10" (id 0) (at 41.91 167.64 0))
     (property "Value" "74LS00" (id 1) (at 41.91 170.18 0))
-    (property "Footprint" "Package_DIP:DIP-14_W7.62mm_LongPads" (id 2) (at 41.91 176.53 0)
+    (property "Footprint" "Package_DIP:DIP-14_W7.62mm" (id 2) (at 41.91 176.53 0)
       (effects (font (size 1.27 1.27)) hide)
     )
@@
       (effects (font (size 1.27 1.27)) (justify left))
     )
-    (property "Footprint" "Package_DIP:DIP-14_W7.62mm_LongPads" (id 2) (at 120.65 167.64 0)
+    (property "Footprint" "Package_DIP:DIP-14_W7.62mm" (id 2) (at 120.65 167.64 0)
       (effects (font (size 1.27 1.27)) hide)
     )
@@
       (effects (font (size 1.27 1.27)) (justify left))
     )
-    (property "Footprint" "Package_DIP:DIP-20_W7.62mm_LongPads" (id 2) (at 124.46 109.22 0)
+    (property "Footprint" "Package_DIP:DIP-20_W7.62mm" (id 2) (at 124.46 109.22 0)
       (effects (font (size 1.27 1.27)) hide)
     )
@@
     (property "Reference" "U8" (id 0) (at 57.15 174.625 0))
     (property "Value" "74LS04" (id 1) (at 57.15 177.165 0))
-    (property "Footprint" "Package_DIP:DIP-14_W7.62mm_LongPads" (id 2) (at 57.15 182.88 0)
+    (property "Footprint" "Package_DIP:DIP-14_W7.62mm" (id 2) (at 57.15 182.88 0)
       (effects (font (size 1.27 1.27)) hide)
     )
@@
     (property "Reference" "U9" (id 0) (at 63.5 99.06 0))
     (property "Value" "74LS08" (id 1) (at 63.5 101.6 0))
-    (property "Footprint" "Package_DIP:DIP-14_W7.62mm_LongPads" (id 2) (at 63.5 106.68 0)
-      (effects (font (size 1.27 1.27)) hide)
-    )
+    (property "Footprint" "Package_DIP:DIP-14_W7.62mm" (id 2) (at 63.5 106.68 0)
+      (effects (font (size 1.27 1.27)) hide)
+    )

Commit message: KiCAD: Added R19 (VCCEnable pullup)
Parts:
- added R19: 4K7, custom_footprints:R_Axial_DIN0207_L6.3mm_D2.0mm_P11.43mm_Horizontal, symbol Device:R
Connections:
- net VCC: now also R19.1
- net nVCCEnable: now also R19.2
Other:
- note added: "Not Fitted"
Changed lines of the file:
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@@
   (junction (at 30.48 35.56) (diameter 0) (color 0 0 0 0)
+  )
+  (junction (at 101.6 135.89) (diameter 0) (color 0 0 0 0)
   )
   (junction (at 55.88 93.98) (diameter 0) (color 0 0 0 0)
@@
     (stroke (width 0) (type default) (color 0 0 0 0))
   )
-  (wire (pts (xy 109.22 125.73) (xy 109.22 121.92))
+  (wire (pts (xy 109.22 135.89) (xy 109.22 121.92))
     (stroke (width 0) (type default) (color 0 0 0 0))
   )
@@
     (stroke (width 0) (type default) (color 0 0 0 0))
   )
+  (wire (pts (xy 101.6 133.35) (xy 101.6 135.89))
+    (stroke (width 0) (type default) (color 0 0 0 0))
+  )
   (bus (pts (xy 93.98 111.76) (xy 93.98 114.3))
     (stroke (width 0) (type default) (color 0 0 0 0))
@@
     (stroke (width 0) (type default) (color 0 0 0 0))
   )
+  (wire (pts (xy 95.25 135.89) (xy 101.6 135.89))
+    (stroke (width 0) (type default) (color 0 0 0 0))
+  )
   (wire (pts (xy 194.31 130.81) (xy 194.31 69.85))
     (stroke (width 0) (type default) (color 0 0 0 0))
@@
     (stroke (width 0) (type default) (color 0 0 0 0))
   )
+  (wire (pts (xy 101.6 135.89) (xy 109.22 135.89))
+    (stroke (width 0) (type default) (color 0 0 0 0))
+  )
   (wire (pts (xy 161.29 96.52) (xy 173.99 96.52))
     (stroke (width 0) (type default) (color 0 0 0 0))
@@
     (stroke (width 0) (type default) (color 0 0 0 0))
   )
-  (wire (pts (xy 102.87 125.73) (xy 109.22 125.73))
-    (stroke (width 0) (type default) (color 0 0 0 0))
-  )
   (wire (pts (xy 109.22 119.38) (xy 111.76 119.38))
     (stroke (width 0) (type default) (color 0 0 0 0))
@@
   (wire (pts (xy 231.14 123.19) (xy 226.06 123.19))
     (stroke (width 0) (type default) (color 0 0 0 0))
+  )
+  (text "Not Fitted" (at 90.17 130.81 0)
+    (effects (font (size 1.27 1.27)) (justify left bottom))
   )
   (label "Addr5" (at 96.52 54.61 0)
@@
     (effects (font (size 1.27 1.27)) (justify right))
   )
-  (hierarchical_label "nVCCEnable" (shape input) (at 102.87 125.73 180)
+  (hierarchical_label "nVCCEnable" (shape input) (at 95.25 135.89 180)
     (effects (font (size 1.27 1.27)) (justify right))
   )
@@
     (pin "1")
   )
+  (symbol (lib_id "Device:R") (at 101.6 129.54 0) (unit 1)
+    (in_bom yes) (on_board yes) (fields_autoplaced)
+    (property "Reference" "R19" (id 0) (at 104.14 128.2699 0)
+      (effects (font (size 1.27 1.27)) (justify left))
+    )
+    (property "Value" "4K7" (id 1) (at 104.14 130.8099 0)
+      (effects (font (size 1.27 1.27)) (justify left))
+    )
+    (property "Footprint" "custom_footprints:R_Axial_DIN0207_L6.3mm_D2.0mm_P11.43mm_Horizontal" (id 2) (at 99.822 129.54 90)
+      (effects (font (size 1.27 1.27)) hide)
+    )
+    (property "Datasheet" "~" (id 3) (at 101.6 129.54 0)
+      (effects (font (size 1.27 1.27)) hide)
+    )
+    (pin "1")
+    (pin "2")
+  )
   (symbol (lib_id "74xx:74LS00") (at 41.91 176.53 0) (unit 4)
     (in_bom yes) (on_board yes) (fields_autoplaced)
@@
       (effects (font (size 1.27 1.27)) hide)
     )
+    (pin "1")
+  )
+  (symbol (lib_id "power:VCC") (at 101.6 125.73 0) (unit 1)
+    (in_bom yes) (on_board yes) (fields_autoplaced)
+    (property "Reference" "#PWR0149" (id 0) (at 101.6 129.54 0)
+      (effects (font (size 1.27 1.27)) hide)
+    )
+    (property "Value" "VCC" (id 1) (at 101.6 120.65 0))
+    (property "Footprint" "" (id 2) (at 101.6 125.73 0)
+      (effects (font (size 1.27 1.27)) hide)
+    )
+    (property "Datasheet" "" (id 3) (at 101.6 125.73 0)
+      (effects (font (size 1.27 1.27)) hide)
+    )
