File: kicad/main_logic.kicad_sch (KiCad schematic)
At the start: 15 parts, among them U10 74LS00, U17 28 PIN ZIF, U3 74LS245, U4 74LS244, U5 74LS244, U8 74LS04, U9 74LS08

Commit message: KiCAD - more silk screen
Parts:
- R4: footprint custom_footprints:R_Axial_DIN0207_L6.3mm_D2.0mm_P11.43mm_Horizontal -> Resistor_THT:R_Axial_DIN0207_L6.3mm_D2.5mm_P10.16mm_Horizontal
- U10, U8, U9: footprint Package_DIP:DIP-14_W7.62mm -> Package_DIP:DIP-14_W7.62mm_Socket
- U3, U4, U5: footprint Package_DIP:DIP-20_W7.62mm -> Package_DIP:DIP-20_W7.62mm_Socket
Changed lines of the file:
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@@
     (property "Reference" "U10" (id 0) (at 78.74 73.66 0))
     (property "Value" "74LS00" (id 1) (at 78.74 76.2 0))
-    (property "Footprint" "Package_DIP:DIP-14_W7.62mm" (id 2) (at 78.74 82.55 0)
+    (property "Footprint" "Package_DIP:DIP-14_W7.62mm_Socket" (id 2) (at 78.74 82.55 0)
       (effects (font (size 1.27 1.27)) hide)
     )
@@
     (property "Reference" "U9" (id 0) (at 41.91 153.67 0))
     (property "Value" "74LS08" (id 1) (at 41.91 156.21 0))
-    (property "Footprint" "Package_DIP:DIP-14_W7.62mm" (id 2) (at 41.91 161.29 0)
+    (property "Footprint" "Package_DIP:DIP-14_W7.62mm_Socket" (id 2) (at 41.91 161.29 0)
       (effects (font (size 1.27 1.27)) hide)
     )
@@
       (effects (font (size 1.27 1.27)) (justify left))
     )
-    (property "Footprint" "Package_DIP:DIP-14_W7.62mm" (id 2) (at 80.01 167.64 0)
+    (property "Footprint" "Package_DIP:DIP-14_W7.62mm_Socket" (id 2) (at 80.01 167.64 0)
       (effects (font (size 1.27 1.27)) hide)
     )
@@
     (property "Reference" "U8" (id 0) (at 57.15 146.685 0))
     (property "Value" "74LS04" (id 1) (at 57.15 149.225 0))
-    (property "Footprint" "Package_DIP:DIP-14_W7.62mm" (id 2) (at 57.15 154.94 0)
+    (property "Footprint" "Package_DIP:DIP-14_W7.62mm_Socket" (id 2) (at 57.15 154.94 0)
       (effects (font (size 1.27 1.27)) hide)
     )
@@
     (property "Reference" "U10" (id 0) (at 63.5 82.55 0))
     (property "Value" "74LS00" (id 1) (at 63.5 85.09 0))
-    (property "Footprint" "Package_DIP:DIP-14_W7.62mm" (id 2) (at 63.5 91.44 0)
+    (property "Footprint" "Package_DIP:DIP-14_W7.62mm_Socket" (id 2) (at 63.5 91.44 0)
       (effects (font (size 1.27 1.27)) hide)
     )
@@
       (effects (font (size 1.27 1.27)) (justify left))
     )
-    (property "Footprint" "Package_DIP:DIP-14_W7.62mm" (id 2) (at 100.33 167.64 0)
+    (property "Footprint" "Package_DIP:DIP-14_W7.62mm_Socket" (id 2) (at 100.33 167.64 0)
       (effects (font (size 1.27 1.27)) hide)
     )
@@
     (property "Reference" "U8" (id 0) (at 48.26 80.645 0))
     (property "Value" "74LS04" (id 1) (at 48.26 83.185 0))
-    (property "Footprint" "Package_DIP:DIP-14_W7.62mm" (id 2) (at 48.26 88.9 0)
+    (property "Footprint" "Package_DIP:DIP-14_W7.62mm_Socket" (id 2) (at 48.26 88.9 0)
       (effects (font (size 1.27 1.27)) hide)
     )
@@
     (property "Reference" "U10" (id 0) (at 63.5 66.04 0))
     (property "Value" "74LS00" (id 1) (at 63.5 68.58 0))
-    (property "Footprint" "Package_DIP:DIP-14_W7.62mm" (id 2) (at 63.5 74.93 0)
+    (property "Footprint" "Package_DIP:DIP-14_W7.62mm_Socket" (id 2) (at 63.5 74.93 0)
       (effects (font (size 1.27 1.27)) hide)
     )
@@
       (effects (font (size 1.27 1.27)) (justify left))
     )
-    (property "Footprint" "Package_DIP:DIP-20_W7.62mm" (id 2) (at 124.46 54.61 0)
+    (property "Footprint" "Package_DIP:DIP-20_W7.62mm_Socket" (id 2) (at 124.46 54.61 0)
       (effects (font (size 1.27 1.27)) hide)
     )
@@
       (effects (font (size 1.27 1.27)) (justify left))
     )
-    (property "Footprint" "Package_DIP:DIP-20_W7.62mm" (id 2) (at 256.54 54.61 0)
+    (property "Footprint" "Package_DIP:DIP-20_W7.62mm_Socket" (id 2) (at 256.54 54.61 0)
       (effects (font (size 1.27 1.27)) hide)
     )
@@
     (property "Reference" "U8" (id 0) (at 57.15 160.655 0))
     (property "Value" "74LS04" (id 1) (at 57.15 163.195 0))
-    (property "Footprint" "Package_DIP:DIP-14_W7.62mm" (id 2) (at 57.15 168.91 0)
+    (property "Footprint" "Package_DIP:DIP-14_W7.62mm_Socket" (id 2) (at 57.15 168.91 0)
       (effects (font (size 1.27 1.27)) hide)
     )
@@
     (property "Reference" "U10" (id 0) (at 41.91 167.64 0))
     (property "Value" "74LS00" (id 1) (at 41.91 170.18 0))
-    (property "Footprint" "Package_DIP:DIP-14_W7.62mm" (id 2) (at 41.91 176.53 0)
+    (property "Footprint" "Package_DIP:DIP-14_W7.62mm_Socket" (id 2) (at 41.91 176.53 0)
       (effects (font (size 1.27 1.27)) hide)
     )
@@
       (effects (font (size 1.27 1.27)) (justify left))
     )
-    (property "Footprint" "Package_DIP:DIP-14_W7.62mm" (id 2) (at 120.65 167.64 0)
+    (property "Footprint" "Package_DIP:DIP-14_W7.62mm_Socket" (id 2) (at 120.65 167.64 0)
       (effects (font (size 1.27 1.27)) hide)
     )
@@
       (effects (font (size 1.27 1.27)) (justify left))
     )
-    (property "Footprint" "Package_DIP:DIP-20_W7.62mm" (id 2) (at 124.46 109.22 0)
+    (property "Footprint" "Package_DIP:DIP-20_W7.62mm_Socket" (id 2) (at 124.46 109.22 0)
       (effects (font (size 1.27 1.27)) hide)
     )
@@
     (property "Reference" "U8" (id 0) (at 57.15 174.625 0))
     (property "Value" "74LS04" (id 1) (at 57.15 177.165 0))
-    (property "Footprint" "Package_DIP:DIP-14_W7.62mm" (id 2) (at 57.15 182.88 0)
+    (property "Footprint" "Package_DIP:DIP-14_W7.62mm_Socket" (id 2) (at 57.15 182.88 0)
       (effects (font (size 1.27 1.27)) hide)
     )
@@
     (property "Reference" "U9" (id 0) (at 63.5 99.06 0))
     (property "Value" "74LS08" (id 1) (at 63.5 101.6 0))
-    (property "Footprint" "Package_DIP:DIP-14_W7.62mm" (id 2) (at 63.5 106.68 0)
+    (property "Footprint" "Package_DIP:DIP-14_W7.62mm_Socket" (id 2) (at 63.5 106.68 0)
       (effects (font (size 1.27 1.27)) hide)
     )
@@
       (effects (font (size 1.27 1.27)) (justify left))
     )
-    (property "Footprint" "custom_footprints:R_Axial_DIN0207_L6.3mm_D2.0mm_P11.43mm_Horizontal" (id 2) (at 159.258 96.52 90)
-      (effects (font (size 1.27 1.27)) hide)
-    )
+    (property "Footprint" "Resistor_THT:R_Axial_DIN0207_L6.3mm_D2.5mm_P10.16mm_Horizontal" (id 2) (at 159.258 96.52 90)
+      (effects (font (size 1.27 1.27)) hide)
+    )

Commit message: KiCAD: Customize IC footprint silk screen
Parts:
- U10, U8, U9: footprint Package_DIP:DIP-14_W7.62mm_Socket -> custom_footprints:DIP-14_W7.62mm_Socket
- U3, U4, U5: footprint Package_DIP:DIP-20_W7.62mm_Socket -> custom_footprints:DIP-20_W7.62mm_Socket
Changed lines of the file:
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@@
     (property "Reference" "U10" (id 0) (at 78.74 73.66 0))
     (property "Value" "74LS00" (id 1) (at 78.74 76.2 0))
-    (property "Footprint" "Package_DIP:DIP-14_W7.62mm_Socket" (id 2) (at 78.74 82.55 0)
+    (property "Footprint" "custom_footprints:DIP-14_W7.62mm_Socket" (id 2) (at 78.74 82.55 0)
       (effects (font (size 1.27 1.27)) hide)
     )
@@
     (property "Reference" "U9" (id 0) (at 41.91 153.67 0))
     (property "Value" "74LS08" (id 1) (at 41.91 156.21 0))
-    (property "Footprint" "Package_DIP:DIP-14_W7.62mm_Socket" (id 2) (at 41.91 161.29 0)
+    (property "Footprint" "custom_footprints:DIP-14_W7.62mm_Socket" (id 2) (at 41.91 161.29 0)
       (effects (font (size 1.27 1.27)) hide)
     )
@@
       (effects (font (size 1.27 1.27)) (justify left))
     )
-    (property "Footprint" "Package_DIP:DIP-14_W7.62mm_Socket" (id 2) (at 80.01 167.64 0)
+    (property "Footprint" "custom_footprints:DIP-14_W7.62mm_Socket" (id 2) (at 80.01 167.64 0)
       (effects (font (size 1.27 1.27)) hide)
     )
@@
     (property "Reference" "U8" (id 0) (at 57.15 146.685 0))
     (property "Value" "74LS04" (id 1) (at 57.15 149.225 0))
-    (property "Footprint" "Package_DIP:DIP-14_W7.62mm_Socket" (id 2) (at 57.15 154.94 0)
+    (property "Footprint" "custom_footprints:DIP-14_W7.62mm_Socket" (id 2) (at 57.15 154.94 0)
       (effects (font (size 1.27 1.27)) hide)
     )
@@
     (property "Reference" "U10" (id 0) (at 63.5 82.55 0))
     (property "Value" "74LS00" (id 1) (at 63.5 85.09 0))
-    (property "Footprint" "Package_DIP:DIP-14_W7.62mm_Socket" (id 2) (at 63.5 91.44 0)
+    (property "Footprint" "custom_footprints:DIP-14_W7.62mm_Socket" (id 2) (at 63.5 91.44 0)
       (effects (font (size 1.27 1.27)) hide)
     )
@@
       (effects (font (size 1.27 1.27)) (justify left))
     )
-    (property "Footprint" "Package_DIP:DIP-14_W7.62mm_Socket" (id 2) (at 100.33 167.64 0)
+    (property "Footprint" "custom_footprints:DIP-14_W7.62mm_Socket" (id 2) (at 100.33 167.64 0)
       (effects (font (size 1.27 1.27)) hide)
     )
@@
     (property "Reference" "U8" (id 0) (at 48.26 80.645 0))
     (property "Value" "74LS04" (id 1) (at 48.26 83.185 0))
-    (property "Footprint" "Package_DIP:DIP-14_W7.62mm_Socket" (id 2) (at 48.26 88.9 0)
+    (property "Footprint" "custom_footprints:DIP-14_W7.62mm_Socket" (id 2) (at 48.26 88.9 0)
       (effects (font (size 1.27 1.27)) hide)
     )
@@
     (property "Reference" "U10" (id 0) (at 63.5 66.04 0))
     (property "Value" "74LS00" (id 1) (at 63.5 68.58 0))
-    (property "Footprint" "Package_DIP:DIP-14_W7.62mm_Socket" (id 2) (at 63.5 74.93 0)
+    (property "Footprint" "custom_footprints:DIP-14_W7.62mm_Socket" (id 2) (at 63.5 74.93 0)
       (effects (font (size 1.27 1.27)) hide)
     )
@@
       (effects (font (size 1.27 1.27)) (justify left))
     )
-    (property "Footprint" "Package_DIP:DIP-20_W7.62mm_Socket" (id 2) (at 124.46 54.61 0)
+    (property "Footprint" "custom_footprints:DIP-20_W7.62mm_Socket" (id 2) (at 124.46 54.61 0)
       (effects (font (size 1.27 1.27)) hide)
     )
@@
       (effects (font (size 1.27 1.27)) (justify left))
     )
-    (property "Footprint" "Package_DIP:DIP-20_W7.62mm_Socket" (id 2) (at 256.54 54.61 0)
+    (property "Footprint" "custom_footprints:DIP-20_W7.62mm_Socket" (id 2) (at 256.54 54.61 0)
       (effects (font (size 1.27 1.27)) hide)
     )
@@
     (property "Reference" "U8" (id 0) (at 57.15 160.655 0))
     (property "Value" "74LS04" (id 1) (at 57.15 163.195 0))
-    (property "Footprint" "Package_DIP:DIP-14_W7.62mm_Socket" (id 2) (at 57.15 168.91 0)
+    (property "Footprint" "custom_footprints:DIP-14_W7.62mm_Socket" (id 2) (at 57.15 168.91 0)
       (effects (font (size 1.27 1.27)) hide)
     )
@@
     (property "Reference" "U10" (id 0) (at 41.91 167.64 0))
     (property "Value" "74LS00" (id 1) (at 41.91 170.18 0))
-    (property "Footprint" "Package_DIP:DIP-14_W7.62mm_Socket" (id 2) (at 41.91 176.53 0)
+    (property "Footprint" "custom_footprints:DIP-14_W7.62mm_Socket" (id 2) (at 41.91 176.53 0)
       (effects (font (size 1.27 1.27)) hide)
     )
@@
       (effects (font (size 1.27 1.27)) (justify left))
     )
-    (property "Footprint" "Package_DIP:DIP-14_W7.62mm_Socket" (id 2) (at 120.65 167.64 0)
+    (property "Footprint" "custom_footprints:DIP-14_W7.62mm_Socket" (id 2) (at 120.65 167.64 0)
       (effects (font (size 1.27 1.27)) hide)
     )
@@
       (effects (font (size 1.27 1.27)) (justify left))
     )
-    (property "Footprint" "Package_DIP:DIP-20_W7.62mm_Socket" (id 2) (at 124.46 109.22 0)
+    (property "Footprint" "custom_footprints:DIP-20_W7.62mm_Socket" (id 2) (at 124.46 109.22 0)
       (effects (font (size 1.27 1.27)) hide)
     )
@@
     (property "Reference" "U8" (id 0) (at 57.15 174.625 0))
     (property "Value" "74LS04" (id 1) (at 57.15 177.165 0))
-    (property "Footprint" "Package_DIP:DIP-14_W7.62mm_Socket" (id 2) (at 57.15 182.88 0)
+    (property "Footprint" "custom_footprints:DIP-14_W7.62mm_Socket" (id 2) (at 57.15 182.88 0)
       (effects (font (size 1.27 1.27)) hide)
     )
@@
     (property "Reference" "U9" (id 0) (at 63.5 99.06 0))
     (property "Value" "74LS08" (id 1) (at 63.5 101.6 0))
-    (property "Footprint" "Package_DIP:DIP-14_W7.62mm_Socket" (id 2) (at 63.5 106.68 0)
-      (effects (font (size 1.27 1.27)) hide)
-    )
+    (property "Footprint" "custom_footprints:DIP-14_W7.62mm_Socket" (id 2) (at 63.5 106.68 0)
+      (effects (font (size 1.27 1.27)) hide)
+    )

Commit message: KiCAD: Use 0.95mm holes for ZIF socket
Parts:
- U17: footprint Package_DIP:DIP-28_W15.24mm_Socket -> custom_footprints:DIP-28_W15.24mm_Socket_LongPads
Changed lines of the file:
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@@
       (effects (font (size 1.27 1.27)) (justify left))
     )
-    (property "Footprint" "Package_DIP:DIP-28_W15.24mm_Socket" (id 2) (at 222.25 64.77 0)
+    (property "Footprint" "custom_footprints:DIP-28_W15.24mm_Socket_LongPads" (id 2) (at 222.25 64.77 0)
       (effects (font (size 1.27 1.27)) hide)
     )
