File: kicad/power_supply.kicad_sch (KiCad schematic)
At the start: 63 parts, among them J2 Cliff DC10A, Q1 2N2905A, Q2 2N2905A, Q3 2N3904, Q4 2N3904, U11 7406, U16 MC34063AP, U18 LM7805, U19 LM317T, U20 LM317T

Commit message: KiCAD: Make space for full ZIF
Connections:
- net EpromVCCUnswitched: now reaches C9.1, Q1.1 (E), R6.1, R7.1, U19.2 (VO)
- net EpromVPPUnswitched: now reaches C16.1, Q2.1 (E), R13.1, R14.1, U20.2 (VO)
Changed lines of the file:
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@@
+    (effects (font (size 1.27 1.27)) (justify left bottom))
+  )
+  (label "EpromVCCUnswitched" (at 207.01 114.3 0)
     (effects (font (size 1.27 1.27)) (justify left bottom))
   )
@@
     (effects (font (size 1.27 1.27)) (justify left bottom))
   )
+  (label "EpromVPPUnswitched" (at 198.12 29.21 0)
+    (effects (font (size 1.27 1.27)) (justify left bottom))
+  )

Commit message: KiCAD: Add 100n close to MC34063A
Parts:
- added C12: 100n, Capacitor_THT:C_Disc_D4.3mm_W1.9mm_P5.00mm, symbol Device:C
- renumbered C12 to C13, C13 to C14, C14 to C15, C15 to C16, C16 to C17
Connections:
- net 9VDC: now also C12.1
- net GND: now also C12.2
Other:
- moved on the sheet: C11

Commit message: KiCAD: silk screen
Other:
- note added: "Left Trimmer: Adjusts 25V VPP"
- note added: "Right Trimmer: Adjusts 12.5V VPP"
- note removed: "Left Trimmer: Adjusts 12.5V VPP"
- note removed: "Right Trimmer: Adjusts 25V VPP"
Changed lines of the file:
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@@
     (stroke (width 0) (type default) (color 0 0 0 0))
   )
-  (text "Right Trimmer:\nAdjusts 25V VPP" (at 160.02 74.93 180)
+  (text "Left Trimmer:\nAdjusts 25V VPP" (at 160.02 74.93 180)
     (effects (font (size 1.27 1.27)) (justify right bottom))
   )
@@
     (effects (font (size 1.27 1.27)) (justify left bottom))
   )
-  (text "Left Trimmer:\nAdjusts 12.5V VPP" (at 156.21 39.37 180)
+  (text "Right Trimmer:\nAdjusts 12.5V VPP" (at 156.21 39.37 180)
     (effects (font (size 1.27 1.27)) (justify right bottom))
   )

Commit message: KiCAD: larger 0R33; silk screen
Parts:
- R20: footprint custom_footprints:R_Axial_DIN0207_L6.3mm_D2.0mm_P10.16mm_Horizontal -> Resistor_THT:R_Axial_DIN0207_L6.3mm_D2.5mm_P10.16mm_Horizontal
Changed lines of the file:
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@@
     (property "Reference" "R20" (id 0) (at 69.85 22.86 90))
     (property "Value" "0R33" (id 1) (at 69.85 25.4 90))
-    (property "Footprint" "custom_footprints:R_Axial_DIN0207_L6.3mm_D2.0mm_P10.16mm_Horizontal" (id 2) (at 69.85 30.988 90)
+    (property "Footprint" "Resistor_THT:R_Axial_DIN0207_L6.3mm_D2.5mm_P10.16mm_Horizontal" (id 2) (at 69.85 30.988 90)
       (effects (font (size 1.27 1.27)) hide)
     )

Commit message: KiCAD: Holes now M3, inset 4.25mm X and 3.7mm Y
Parts:
- H1, H2, H3, H4: footprint MountingHole:MountingHole_2.7mm_M2.5 -> MountingHole:MountingHole_3.2mm_M3
Changed lines of the file:
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@@
       (effects (font (size 1.27 1.27)) (justify left))
     )
-    (property "Footprint" "MountingHole:MountingHole_2.7mm_M2.5" (id 2) (at 25.4 165.1 0)
+    (property "Footprint" "MountingHole:MountingHole_3.2mm_M3" (id 2) (at 25.4 165.1 0)
       (effects (font (size 1.27 1.27)) hide)
     )
@@
       (effects (font (size 1.27 1.27)) (justify left))
     )
-    (property "Footprint" "MountingHole:MountingHole_2.7mm_M2.5" (id 2) (at 25.4 177.8 0)
+    (property "Footprint" "MountingHole:MountingHole_3.2mm_M3" (id 2) (at 25.4 177.8 0)
       (effects (font (size 1.27 1.27)) hide)
     )
@@
       (effects (font (size 1.27 1.27)) (justify left))
     )
-    (property "Footprint" "MountingHole:MountingHole_2.7mm_M2.5" (id 2) (at 50.8 165.1 0)
+    (property "Footprint" "MountingHole:MountingHole_3.2mm_M3" (id 2) (at 50.8 165.1 0)
       (effects (font (size 1.27 1.27)) hide)
     )
@@
       (effects (font (size 1.27 1.27)) (justify left))
     )
-    (property "Footprint" "MountingHole:MountingHole_2.7mm_M2.5" (id 2) (at 50.8 177.8 0)
-      (effects (font (size 1.27 1.27)) hide)
-    )
+    (property "Footprint" "MountingHole:MountingHole_3.2mm_M3" (id 2) (at 50.8 177.8 0)
+      (effects (font (size 1.27 1.27)) hide)
+    )
